Commit message: Rename finger_left to left_finger

File: onrobot_3fg15_gripper_description/urdf/onrobot_3fg15_gripper.urdf.xacro (robot description, xacro)
@@ -55,5 +55,5 @@
         </xacro:macro>
         <!-- FINGER UPPER -->
-        <joint name="${prefix}_finger_upper_joint" type="revolute">
+        <joint name="${prefix}_upper_finger_joint" type="revolute">
             <limit lower="0" upper="2.86775049" effort="1.0" velocity="0.6"/>
             <axis xyz="1 0 0"/>
@@ -69,5 +69,5 @@
                 <motorTorqueConstant>1</motorTorqueConstant>
             </actuator>
-            <joint name="${prefix}_finger_upper_joint" >
+            <joint name="${prefix}_upper_finger_joint" >
                 <hardwareInterface>hardware_interface/PositionJointInterface</hardwareInterface>
             </joint>
@@ -103,5 +103,5 @@
         </gazebo>
          <!-- THUMB UPPER -->
-        <joint name="${prefix}_thumb_upper_joint" type="fixed">
+        <joint name="${prefix}_upper_thumb_joint" type="fixed">
             <xacro:if value="${position == 1}">
                 <origin xyz="0.0095 0 0.0135" rpy="0.0 0.0 0" />
@@ -146,5 +146,5 @@
         </gazebo>
         <!-- FINGER LEFT -->
-        <joint name="${prefix}_finger_left_joint" type="revolute">
+        <joint name="${prefix}_left_finger_joint" type="revolute">
             <limit lower="0" upper="2.86775049" effort="1.0" velocity="0.6"/>
             <axis xyz="1 0 0"/>
@@ -153,8 +153,8 @@
             <child link="${prefix}_left_finger" />
             <dynamics damping="0" friction="0"/>
-            <mimic joint="${prefix}_finger_upper_joint" multiplier="1.0" offset="0"/>
-        </joint>
-        <xacro:mimic_joint_plugin_gazebo parent_joint="${prefix}_finger_upper_joint"
-                                         mimic_joint="${prefix}_finger_left_joint" has_pid="false" multiplier="1.0" max_effort="10.0" />
+            <mimic joint="${prefix}_upper_finger_joint" multiplier="1.0" offset="0"/>
+        </joint>
+        <xacro:mimic_joint_plugin_gazebo parent_joint="${prefix}_upper_finger_joint"
+                                         mimic_joint="${prefix}_left_finger_joint" has_pid="false" multiplier="1.0" max_effort="10.0" />
         <link name="${prefix}_left_finger">
             <inertial>
@@ -187,5 +187,5 @@
         </gazebo>
          <!-- THUMB LEFT -->
-        <joint name="${prefix}_thumb_left_joint" type="fixed">
+        <joint name="${prefix}_left_thumb_joint" type="fixed">
             <xacro:if value="${position == 1}">
                 <origin xyz="0.0095 0 0.0135" rpy="0.0 0.0 0" />
@@ -230,5 +230,5 @@
         </gazebo>
         <!-- FINGER RIGHT -->
-        <joint name="${prefix}_finger_right_joint" type="revolute">
+        <joint name="${prefix}_right_finger_joint" type="revolute">
             <limit lower="0" upper="2.86775049" effort="1.0" velocity="0.6"/>
             <axis xyz="1 0 0"/>
@@ -237,8 +237,8 @@
             <child link="${prefix}_right_finger" />
             <dynamics damping="0" friction="0"/>
-            <mimic joint="${prefix}_finger_upper_joint" multiplier="1.0" offset="0"/>
-        </joint>
-        <xacro:mimic_joint_plugin_gazebo parent_joint="${prefix}_finger_upper_joint"
-                                         mimic_joint="${prefix}_finger_right_joint" has_pid="false" multiplier="1.0" max_effort="10.0" />
+            <mimic joint="${prefix}_upper_finger_joint" multiplier="1.0" offset="0"/>
+        </joint>
+        <xacro:mimic_joint_plugin_gazebo parent_joint="${prefix}_upper_finger_joint"
+                                         mimic_joint="${prefix}_right_finger_joint" has_pid="false" multiplier="1.0" max_effort="10.0" />
         <link name="${prefix}_right_finger">
             <inertial>
@@ -271,5 +271,5 @@
         </gazebo>
          <!-- THUMB RIGHT -->
-        <joint name="${prefix}_thumb_right_joint" type="fixed">
+        <joint name="${prefix}_right_thumb_joint" type="fixed">
             <xacro:if value="${position == 1}">
                 <origin xyz="0.0095 0 0.0135" rpy="0.0 0.0 0" />

Commit message: added attacher gazebo plugin to simulate contacts

File: onrobot_3fg15_gripper_description/urdf/onrobot_3fg15_gripper.urdf.xacro (robot description, xacro)
@@ -11,7 +11,7 @@
         <link name="${prefix}_base_link">
             <inertial>
-                <mass value="0.25" />
-                <origin xyz="0 0 0" />
-                <inertia  ixx="1.0" ixy="0.0"  ixz="0.0"  iyy="1.0"  iyz="0.0"  izz="1.0" />
+                <mass value="0.95" />
+                <origin xyz="0 0 0" />
+                <inertia  ixx="0.004541317" ixy="0.0"  ixz="0.0"  iyy="0.004541317"  iyz="0.0"  izz="0.003952633" />
             </inertial>
             <visual>
@@ -36,5 +36,29 @@
             <turnGravityOff>false</turnGravityOff>
         </gazebo>
-        <xacro:macro name="mimic_joint_plugin_gazebo" params="parent_joint mimic_joint has_pid:=false multiplier:=1.0 offset:=0 sensitiveness:=0.0 max_effort:=1.0 robot_namespace:=''">
+        <joint name="${prefix}contact_joint" type="prismatic">
+            <limit lower="0" upper="0.00001" effort="1.0" velocity="0.00001"/>
+            <origin xyz="0.0 0 0.18" rpy="0 0 0" />
+            <parent link="${prefix}_base_link"/>
+            <child link="${prefix}contact_link"/>
+        </joint>
+        <!-- BASE LINK -->
+        <link name="${prefix}contact_link">
+            <inertial>
+                <mass value="0.095" />
+                <origin xyz="0 0 0" />
+                <inertia  ixx="0.0004541317" ixy="0.0"  ixz="0.0"  iyy="0.0004541317"  iyz="0.0"  izz="0.0003952633" />
+            </inertial>
+        </link>
+        <transmission name="${prefix}contact_joint">
+            <type>transmission_interface/SimpleTransmission</type>
+            <actuator name="${prefix}contact_joint_motor">
+                <mechanicalReduction>1</mechanicalReduction>
+                <motorTorqueConstant>1</motorTorqueConstant>
+            </actuator>
+            <joint name="${prefix}contact_joint" >
+                <hardwareInterface>hardware_interface/PositionJointInterface</hardwareInterface>
+            </joint>
+        </transmission>
+<!--         <xacro:macro name="mimic_joint_plugin_gazebo" params="parent_joint mimic_joint has_pid:=false multiplier:=1.0 offset:=0 sensitiveness:=0.0 max_effort:=1.0 robot_namespace:=''">
             <gazebo>
                 <plugin name="${mimic_joint}_mimic_joint_plugin" filename="libroboticsgroup_gazebo_mimic_joint_plugin.so">
@@ -53,7 +77,17 @@
                 </plugin>
             </gazebo>
+        </xacro:macro> -->
+        <xacro:macro name="ros_link_attacher_plugin">
+          <gazebo>
+            <plugin name="ros_link_attacher_plugin" filename="libgazebo_ros_link_attacher.so"/>"
+          </gazebo>
         </xacro:macro>
+        <joint name="${prefix}_upper_finger_joint" type="fixed">
+            <origin xyz="0.1022 0.0 -0.03" rpy="0.0 0.0 0.0" />
+            <parent link="${prefix}_base_link"/>
+            <child link="${prefix}_upper_finger" />
+        </joint>
         <!-- FINGER UPPER -->
-        <joint name="${prefix}_upper_finger_joint" type="revolute">
+        <!--joint name="${prefix}_upper_finger_joint" type="revolute">
             <limit lower="0" upper="2.86775049" effort="1.0" velocity="0.6"/>
             <axis xyz="1 0 0"/>
@@ -72,12 +106,12 @@
                 <hardwareInterface>hardware_interface/PositionJointInterface</hardwareInterface>
             </joint>
-        </transmission>
+        </transmission-->
         <link name="${prefix}_upper_finger">
             <inertial>
-                <mass value="0.1" />
-                <origin xyz="0 0 0" />
-            <inertia ixx="1.0" ixy="0.0" ixz="0.0"
-                    iyy="1.0" iyz="0.0"
-                    izz="1.0" />
+                <mass value="0.003333" />
+                <origin xyz="0 0 0" />
+            <inertia ixx="0.000000277" ixy="0.0" ixz="0.0"
+                    iyy="0.000000277" iyz="0.0"
+                    izz="0.000000056" />
             </inertial>
             <visual>
@@ -118,9 +152,9 @@
         <link name="${prefix}_upper_thumb">
             <inertial>
-                <mass value="0.1" />
-                <origin xyz="0 0 0" />
-            <inertia ixx="1.0" ixy="0.0" ixz="0.0"
-                    iyy="1.0" iyz="0.0"
-                    izz="1.0" />
+                <mass value="0.0033333" />
+                <origin xyz="0 0 0" />
+            <inertia ixx="0.000000277" ixy="0.0" ixz="0.0"
+                    iyy="0.000000277" iyz="0.0"
+                    izz="0.000000056" />
             </inertial>
             <visual>
@@ -145,6 +179,11 @@
             <turnGravityOff>false</turnGravityOff>
         </gazebo>
+        <joint name="${prefix}_left_finger_joint" type="fixed">
+            <origin xyz="0.1022 0.02598 0.015" rpy="2.0944 0 0" />
+            <parent link="${prefix}_base_link"/>
+            <child link="${prefix}_left_finger" />
+        </joint>
         <!-- FINGER LEFT -->
-        <joint name="${prefix}_left_finger_joint" type="revolute">
+        <!--joint name="${prefix}_left_finger_joint" type="revolute">
             <limit lower="0" upper="2.86775049" effort="1.0" velocity="0.6"/>
             <axis xyz="1 0 0"/>
@@ -156,12 +195,12 @@
         </joint>
         <xacro:mimic_joint_plugin_gazebo parent_joint="${prefix}_upper_finger_joint"
-                                         mimic_joint="${prefix}_left_finger_joint" has_pid="false" multiplier="1.0" max_effort="10.0" />
+                                         mimic_joint="${prefix}_left_finger_joint" has_pid="false" multiplier="1.0" max_effort="10.0" /-->
         <link name="${prefix}_left_finger">
             <inertial>
-                <mass value="0.1" />
-                <origin xyz="0 0 0" />
-            <inertia ixx="1.0" ixy="0.0" ixz="0.0"
-                    iyy="1.0" iyz="0.0"
-                    izz="1.0" />
+                <mass value="0.0033333" />
+                <origin xyz="0 0 0" />
+            <inertia ixx="0.000000277" ixy="0.0" ixz="0.0"
+                    iyy="0.000000277" iyz="0.0"
+                    izz="0.000000056" />
             </inertial>
             <visual>
@@ -202,9 +241,9 @@
         <link name="${prefix}_left_thumb">
             <inertial>
-                <mass value="0.1" />
-                <origin xyz="0 0 0" />
-            <inertia ixx="1.0" ixy="0.0" ixz="0.0"
-                    iyy="1.0" iyz="0.0"
-                    izz="1.0" />
+                <mass value="0.00333" />
+                <origin xyz="0 0 0" />
+            <inertia ixx="0.000000277" ixy="0.0" ixz="0.0"
+                    iyy="0.000000277" iyz="0.0"
+                    izz="0.000000056" />
             </inertial>
             <visual>
@@ -229,6 +268,11 @@
             <turnGravityOff>false</turnGravityOff>
         </gazebo>
+        <joint name="${prefix}_right_finger_joint" type="fixed">
+            <origin xyz="0.1022 -0.02598 0.015" rpy="-2.0944 0 0" />
+            <parent link="${prefix}_base_link"/>
+            <child link="${prefix}_right_finger" />
+        </joint>
         <!-- FINGER RIGHT -->
-        <joint name="${prefix}_right_finger_joint" type="revolute">
+        <!--joint name="${prefix}_right_finger_joint" type="revolute">
             <limit lower="0" upper="2.86775049" effort="1.0" velocity="0.6"/>
             <axis xyz="1 0 0"/>
@@ -240,12 +284,12 @@
         </joint>
         <xacro:mimic_joint_plugin_gazebo parent_joint="${prefix}_upper_finger_joint"
-                                         mimic_joint="${prefix}_right_finger_joint" has_pid="false" multiplier="1.0" max_effort="10.0" />
+                                         mimic_joint="${prefix}_right_finger_joint" has_pid="false" multiplier="1.0" max_effort="10.0" /-->
         <link name="${prefix}_right_finger">
             <inertial>
-                <mass value="0.1" />
-                <origin xyz="0 0 0" />
-            <inertia ixx="1.0" ixy="0.0" ixz="0.0"
-                    iyy="1.0" iyz="0.0"
-                    izz="1.0" />
+                <mass value="0.003333" />
+                <origin xyz="0 0 0" />
+            <inertia ixx="0.000000277" ixy="0.0" ixz="0.0"
+                    iyy="0.000000277" iyz="0.0"
+                    izz="0.000000056" />
             </inertial>
             <visual>
@@ -286,9 +330,9 @@
         <link name="${prefix}_right_thumb">
             <inertial>
-                <mass value="0.1" />
-                <origin xyz="0 0 0" />
-            <inertia ixx="1.0" ixy="0.0" ixz="0.0"
-                    iyy="1.0" iyz="0.0"
-                    izz="1.0" />
+                <mass value="0.0033333" />
+                <origin xyz="0 0 0" />
+            <inertia ixx="0.000000277" ixy="0.0" ixz="0.0"
+                    iyy="0.000000277" iyz="0.0"
+                    izz="0.000000056" />
             </inertial>
             <visual>

Commit message: fast fix to add missing xacro tag

File: onrobot_3fg15_gripper_description/urdf/onrobot_3fg15_gripper.urdf.xacro (robot description, xacro)
@@ -4,5 +4,5 @@
     <xacro:macro name="onrobot_3fg15_gripper" params="prefix parent *origin position:=2">
         <joint name="${prefix}_base_joint" type="fixed">
-            <insert_block name="origin"/>
+            <xacro:insert_block name="origin" />
             <parent link="${parent}"/>
             <child link="${prefix}_base_link"/>
@@ -34,4 +34,52 @@
         <gazebo reference="${prefix}_base_link">
             <material>Gazebo/Grey</material>
+            <turnGravityOff>false</turnGravityOff>
+        </gazebo>
+        <!-- FINGER UPPER -->
+        <joint name="${prefix}_upper_finger_joint" type="revolute">
+            <limit lower="0" upper="2.86775049" effort="1.0" velocity="0.6"/>
+            <axis xyz="1 0 0"/>
+            <origin xyz="0.1022 0.0 -0.03" rpy="0.0 0.0 0.0" />
+            <parent link="${prefix}_base_link"/>
+            <child link="${prefix}_upper_finger" />
+            <dynamics damping="0" friction="0"/>
+        </joint>
+        <transmission name="${prefix}_base_trans_upper">
+            <type>transmission_interface/SimpleTransmission</type>
+            <actuator name="${prefix}_base_motor_upper">
+                <mechanicalReduction>1</mechanicalReduction>
+                <motorTorqueConstant>1</motorTorqueConstant>
+            </actuator>
+            <joint name="${prefix}_upper_finger_joint" >
+                <hardwareInterface>hardware_interface/PositionJointInterface</hardwareInterface>
+            </joint>
+        </transmission>
+        <link name="${prefix}_upper_finger">
+            <inertial>
+                <mass value="0.1" />
+                <origin xyz="0 0 0" />
+            <inertia ixx="1.0" ixy="0.0" ixz="0.0"
+                    iyy="1.0" iyz="0.0"
+                    izz="1.0" />
+            </inertial>
+            <visual>
+                <origin xyz="0.0 0 0" rpy="0 0 0" />
+                <geometry>
+                    <mesh filename="package://onrobot_3fg15_gripper_description/meshes/onrobot_3fg15_finger.stl" scale="1.0 1.0 1.0"/>
+                </geometry>
+                <material name="black">
+                <color rgba="0.2 0.2 0.2 1"/>
+                </material>
+            </visual>
+            <collision>
+                <origin xyz="0 0 0" rpy="0 0 0" />
+                <geometry>
+                    <mesh filename="package://onrobot_3fg15_gripper_description/meshes/onrobot_3fg15_finger.stl" scale="1.0 1.0 1.0"/>
+                </geometry>
+            </collision>
+            <contact_coefficients kd="1.0" kp="1000.0" mu="0"/>
+        </link>
+        <gazebo reference="${prefix}_upper_finger">
+            <material>Gazebo/White</material>
             <turnGravityOff>false</turnGravityOff>
         </gazebo>
@@ -54,52 +102,4 @@
             </gazebo>
         </xacro:macro>
-        <!-- FINGER UPPER -->
-        <joint name="${prefix}_upper_finger_joint" type="revolute">
-            <limit lower="0" upper="2.86775049" effort="1.0" velocity="0.6"/>
-            <axis xyz="1 0 0"/>
-            <origin xyz="0.1022 0.0 -0.03" rpy="0.0 0.0 0.0" />
-            <parent link="${prefix}_base_link"/>
-            <child link="${prefix}_upper_finger" />
-            <dynamics damping="0" friction="0"/>
-        </joint>
-        <transmission name="${prefix}_base_trans_upper">
-            <type>transmission_interface/SimpleTransmission</type>
-            <actuator name="${prefix}_base_motor_upper">
-                <mechanicalReduction>1</mechanicalReduction>
-                <motorTorqueConstant>1</motorTorqueConstant>
-            </actuator>
-            <joint name="${prefix}_upper_finger_joint" >
-                <hardwareInterface>hardware_interface/PositionJointInterface</hardwareInterface>
-            </joint>
-        </transmission>
-        <link name="${prefix}_upper_finger">
-            <inertial>
-                <mass value="0.1" />
-                <origin xyz="0 0 0" />
-            <inertia ixx="1.0" ixy="0.0" ixz="0.0"
-                    iyy="1.0" iyz="0.0"
-                    izz="1.0" />
-            </inertial>
-            <visual>
-                <origin xyz="0.0 0 0" rpy="0 0 0" />
-                <geometry>
-                    <mesh filename="package://onrobot_3fg15_gripper_description/meshes/onrobot_3fg15_finger.stl" scale="1.0 1.0 1.0"/>
-                </geometry>
-                <material name="black">
-                <color rgba="0.2 0.2 0.2 1"/>
-                </material>
-            </visual>
-            <collision>
-                <origin xyz="0 0 0" rpy="0 0 0" />
-                <geometry>
-                    <mesh filename="package://onrobot_3fg15_gripper_description/meshes/onrobot_3fg15_finger.stl" scale="1.0 1.0 1.0"/>
-                </geometry>
-            </collision>
-            <contact_coefficients kd="1.0" kp="1000.0" mu="0"/>
-        </link>
-        <gazebo reference="${prefix}_upper_finger">
-            <material>Gazebo/White</material>
-            <turnGravityOff>false</turnGravityOff>
-        </gazebo>
          <!-- THUMB UPPER -->
         <joint name="${prefix}_upper_thumb_joint" type="fixed">
